File: assets/Boards/Main/Main.kicad_pcb (KiCad board)
At the start: 2 copper layers, 76.2 x 29.2 mm, 16 parts, among them J1 PWR, J2 CTRLS_BOARD, U1 DFRobot_MAX98357, U2 Waveshare_ESP32-S3-Tiny

Commit message: Updated boards.
Routing:
- net SPEAKER_DATA: track 25.7 -> 26.7 mm
Changed lines of the file:
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@@
-	)
-	(segment
-		(start 141.43324 67.668)
-		(end 140.78324 68.318)
-		(width 0.3)
-		(layer "F.Cu")
-		(net 28)
 	)
 	(segment
 		(start 128.577479 72.644)
 		(end 126.746 72.644)
-		(width 0.3)
-		(layer "F.Cu")
-		(net 28)
-	)
-	(segment
-		(start 143.51 66.279)
-		(end 142.121 67.668)
 		(width 0.3)
 		(layer "F.Cu")
@@
 	)
 	(segment
-		(start 142.121 67.668)
-		(end 141.43324 67.668)
-		(width 0.3)
-		(layer "F.Cu")
-		(net 28)
-	)
-	(segment
-		(start 140.78324 68.318)
-		(end 132.90348 68.318)
+		(start 132.90348 68.318)
+		(end 139.639521 68.318)
 		(width 0.3)
 		(layer "F.Cu")
@@
 	)
 	(segment
-		(start 124.707 72.143)
-		(end 122.555 74.295)
+		(start 139.639521 68.318)
+		(end 141.678521 66.279)
 		(width 0.3)
 		(layer "F.Cu")
-		(net 29)
+		(net 28)
 	)
 	(segment
-		(start 142.121 65.128)
-		(end 141.43324 65.128)
+		(start 141.678521 66.279)
+		(end 143.51 66.279)
+		(width 0.3)
+		(layer "F.Cu")
+		(net 28)
+	)
+	(segment
+		(start 124.707 72.143)
+		(end 128.36996 72.143)
 		(width 0.3)
 		(layer "F.Cu")
@@
 	(segment
 		(start 128.36996 72.143)
-		(end 124.707 72.143)
+		(end 132.695959 67.817)
+		(width 0.3)
+		(layer "F.Cu")
+		(net 29)
+	)
+	(segment
+		(start 140.462 64.516)
+		(end 141.239 63.739)
+		(width 0.3)
+		(layer "F.Cu")
+		(net 29)
+	)
+	(segment
+		(start 132.695959 67.817)
+		(end 139.432 67.817)
+		(width 0.3)
+		(layer "F.Cu")
+		(net 29)
+	)
+	(segment
+		(start 141.239 63.739)
+		(end 143.51 63.739)
+		(width 0.3)
+		(layer "F.Cu")
+		(net 29)
+	)
+	(segment
+		(start 140.462 66.787)
+		(end 140.462 64.516)
 		(width 0.3)
 		(layer "F.Cu")
@@
 	(segment
 		(start 139.432 67.817)
-		(end 132.695959 67.817)
+		(end 140.462 66.787)
 		(width 0.3)
 		(layer "F.Cu")
@@
 	)
 	(segment
-		(start 140.759 65.80224)
-		(end 140.759 66.49)
+		(start 122.555 74.295)
+		(end 124.707 72.143)
 		(width 0.3)
 		(layer "F.Cu")
-		(net 29)
-	)
-	(segment
-		(start 141.43324 65.128)
-		(end 140.759 65.80224)
-		(width 0.3)
-		(layer "F.Cu")
-		(net 29)
-	)
-	(segment
-		(start 132.695959 67.817)
-		(end 128.36996 72.143)
-		(width 0.3)
-		(layer "F.Cu")
-		(net 29)
-	)
-	(segment
-		(start 143.51 63.739)
-		(end 142.121 65.128)
-		(width 0.3)
-		(layer "F.Cu")
-		(net 29)
-	)
-	(segment
-		(start 140.759 66.49)
-		(end 139.432 67.817)
-		(width 0.3)
-		(layer "F.Cu")
